File: power_monitor/power_monitor.kicad_pcb (KiCad board)
At the start: 2 copper layers, 60 x 62 mm, 22 parts, among them J1 230V AC Input, J2 230V AC Output, J3 RFID, J4 OLED, J5 WS2812, K1 G2RL-2A-DC5, Q1 FDN339AN, U1 Wemos-D1-mini, U2 ACS723xMATR-10AB

Commit message: Reworked isolation, pours and silkscreen
Routing:
- net +5V: track 140.3 -> 150.2 mm
- net SDA: track 54.1 -> 59.4 mm, vias 0 -> 1
- net WS2812: track 29.3 -> 24.5 mm, vias 0 -> 1
- net Relay: track 30.1 -> 28.2 mm
- net /Power Handling/AC_N_Switched: track 14.0 -> 15.7 mm
- net SCL: track 48.2 -> 46.8 mm
Other:
- board text added: "number here"
